Commit message: made into right arm

File: xacro/gummi.srdf.xacro (robot description, xacro)
@@ -12,6 +12,6 @@
   <!--SUBGROUPS: Groups can also be formed by referencing to already defined group names-->
   <!-- Including the xacro files from base and end effector that containg the macros for each part of the srdf -->
-  <xacro:include filename="$(arg base)/xacro/gummi_base.srdf.xacro" />
-  <xacro:include filename="$(arg ee)/xacro/gummi_ee.srdf.xacro" />
+  <xacro:include filename="$(env GUMMI_RIGHTBASEPATH)/xacro/gummi_base.srdf.xacro" />
+  <xacro:include filename="$(env GUMMI_RIGHTEEPATH)/xacro/gummi_ee.srdf.xacro" />
     <group name="right_arm">
       <xacro:group_right_arm_base />

File: xacro/gummi_description.urdf.xacro (robot description, xacro)
@@ -2,5 +2,5 @@
 <robot
   name="gummi" xmlns:xacro="http://www.ros.org/wiki/xacro">
-<xacro:include filename="$(arg base)/xacro/gummi_description_base.urdf.xacro" />
-<xacro:include filename="$(arg ee)/xacro/gummi_description_ee.urdf.xacro" />
+<xacro:include filename="$(env GUMMI_RIGHTBASEPATH)/xacro/gummi_description_base.urdf.xacro" />
+<xacro:include filename="$(env GUMMI_RIGHTEEPATH)/xacro/gummi_description_ee.urdf.xacro" />
 </robot>

File: xacro/gummi_description_base.urdf.xacro (robot description, xacro)
@@ -23,5 +23,5 @@
       <geometry>
         <mesh
-          filename="package://gummi_base_$(env ROS_GUMMI_BASE)/meshes/base_link.STL" />
+          filename="package://gummi_rightbase_$(env ROS_GUMMI_RIGHTBASE)/meshes/base_link.STL" />
       </geometry>
       <material
@@ -37,5 +37,5 @@
       <geometry>
         <mesh
-          filename="package://gummi_base_$(env ROS_GUMMI_BASE)/meshes/base_link.STL" />
+          filename="package://gummi_rightbase_$(env ROS_GUMMI_RIGHTBASE)/meshes/base_link.STL" />
       </geometry>
     </collision>
@@ -63,19 +63,19 @@
       <geometry>
         <mesh
-          filename="package://gummi_base_$(env ROS_GUMMI_BASE)/meshes/shoulder_preroll.STL" />
-      </geometry>
-      <material
-        name="">
-        <color
-          rgba="0.79216 0.81961 0.93333 1" />
-      </material>
-    </visual>
-    <collision>
-      <origin
-        xyz="0 0 0"
-        rpy="0 0 0" />
-      <geometry>
-        <mesh
-          filename="package://gummi_base_$(env ROS_GUMMI_BASE)/meshes/shoulder_preroll.STL" />
+          filename="package://gummi_rightbase_$(env ROS_GUMMI_RIGHTBASE)/meshes/shoulder_preroll.STL" />
+      </geometry>
+      <material
+        name="">
+        <color
+          rgba="0.79216 0.81961 0.93333 1" />
+      </material>
+    </visual>
+    <collision>
+      <origin
+        xyz="0 0 0"
+        rpy="0 0 0" />
+      <geometry>
+        <mesh
+          filename="package://gummi_rightbase_$(env ROS_GUMMI_RIGHTBASE)/meshes/shoulder_preroll.STL" />
       </geometry>
     </collision>
@@ -121,19 +121,19 @@
       <geometry>
         <mesh
-          filename="package://gummi_base_$(env ROS_GUMMI_BASE)/meshes/shoulder.STL" />
-      </geometry>
-      <material
-        name="">
-        <color
-          rgba="0.79216 0.81961 0.93333 1" />
-      </material>
-    </visual>
-    <collision>
-      <origin
-        xyz="0 0 0"
-        rpy="0 0 0" />
-      <geometry>
-        <mesh
-          filename="package://gummi_base_$(env ROS_GUMMI_BASE)/meshes/shoulder.STL" />
+          filename="package://gummi_rightbase_$(env ROS_GUMMI_RIGHTBASE)/meshes/shoulder.STL" />
+      </geometry>
+      <material
+        name="">
+        <color
+          rgba="0.79216 0.81961 0.93333 1" />
+      </material>
+    </visual>
+    <collision>
+      <origin
+        xyz="0 0 0"
+        rpy="0 0 0" />
+      <geometry>
+        <mesh
+          filename="package://gummi_rightbase_$(env ROS_GUMMI_RIGHTBASE)/meshes/shoulder.STL" />
       </geometry>
     </collision>
@@ -179,19 +179,19 @@
       <geometry>
         <mesh
-          filename="package://gummi_base_$(env ROS_GUMMI_BASE)/meshes/upperarm_preroll.STL" />
-      </geometry>
-      <material
-        name="">
-        <color
-          rgba="0.79216 0.81961 0.93333 1" />
-      </material>
-    </visual>
-    <collision>
-      <origin
-        xyz="0 0 0"
-        rpy="0 0 0" />
-      <geometry>
-        <mesh
-          filename="package://gummi_base_$(env ROS_GUMMI_BASE)/meshes/upperarm_preroll.STL" />
+          filename="package://gummi_rightbase_$(env ROS_GUMMI_RIGHTBASE)/meshes/upperarm_preroll.STL" />
+      </geometry>
+      <material
+        name="">
+        <color
+          rgba="0.79216 0.81961 0.93333 1" />
+      </material>
+    </visual>
+    <collision>
+      <origin
+        xyz="0 0 0"
+        rpy="0 0 0" />
+      <geometry>
+        <mesh
+          filename="package://gummi_rightbase_$(env ROS_GUMMI_RIGHTBASE)/meshes/upperarm_preroll.STL" />
       </geometry>
     </collision>
@@ -237,19 +237,19 @@
       <geometry>
         <mesh
-          filename="package://gummi_base_$(env ROS_GUMMI_BASE)/meshes/upperarm.STL" />
-      </geometry>
-      <material
-        name="">
-        <color
-          rgba="0.79216 0.81961 0.93333 1" />
-      </material>
-    </visual>
-    <collision>
-      <origin
-        xyz="0 0 0"
-        rpy="0 0 0" />
-      <geometry>
-        <mesh
-          filename="package://gummi_base_$(env ROS_GUMMI_BASE)/meshes/upperarm.STL" />
+          filename="package://gummi_rightbase_$(env ROS_GUMMI_RIGHTBASE)/meshes/upperarm.STL" />
+      </geometry>
+      <material
+        name="">
+        <color
+          rgba="0.79216 0.81961 0.93333 1" />
+      </material>
+    </visual>
+    <collision>
+      <origin
+        xyz="0 0 0"
+        rpy="0 0 0" />
+      <geometry>
+        <mesh
+          filename="package://gummi_rightbase_$(env ROS_GUMMI_RIGHTBASE)/meshes/upperarm.STL" />
       </geometry>
     </collision>
@@ -295,19 +295,19 @@
       <geometry>
         <mesh
-          filename="package://gummi_base_$(env ROS_GUMMI_BASE)/meshes/lowerarm_preroll_u.STL" />
-      </geometry>
-      <material
-        name="">
-        <color
-          rgba="0.79216 0.81961 0.93333 1" />
-      </material>
-    </visual>
-    <collision>
-      <origin
-        xyz="0 0 0"
-        rpy="0 0 0" />
-      <geometry>
-        <mesh
-          filename="package://gummi_base_$(env ROS_GUMMI_BASE)/meshes/lowerarm_preroll_u.STL" />
+          filename="package://gummi_rightbase_$(env ROS_GUMMI_RIGHTBASE)/meshes/lowerarm_preroll_u.STL" />
+      </geometry>
+      <material
+        name="">
+        <color
+          rgba="0.79216 0.81961 0.93333 1" />
+      </material>
+    </visual>
+    <collision>
+      <origin
+        xyz="0 0 0"
+        rpy="0 0 0" />
+      <geometry>
+        <mesh
+          filename="package://gummi_rightbase_$(env ROS_GUMMI_RIGHTBASE)/meshes/lowerarm_preroll_u.STL" />
       </geometry>
     </collision>
@@ -353,19 +353,19 @@
       <geometry>
         <mesh
-          filename="package://gummi_base_$(env ROS_GUMMI_BASE)/meshes/upperarm_biceps_pulley.STL" />
-      </geometry>
-      <material
-        name="">
-        <color
-          rgba="0.79216 0.81961 0.93333 1" />
-      </material>
-    </visual>
-    <collision>
-      <origin
-        xyz="0 0 0"
-        rpy="0 0 0" />
-      <geometry>
-        <mesh
-          filename="package://gummi_base_$(env ROS_GUMMI_BASE)/meshes/upperarm_biceps_pulley.STL" />
+          filename="package://gummi_rightbase_$(env ROS_GUMMI_RIGHTBASE)/meshes/upperarm_biceps_pulley.STL" />
+      </geometry>
+      <material
+        name="">
+        <color
+          rgba="0.79216 0.81961 0.93333 1" />
+      </material>
+    </visual>
+    <collision>
+      <origin
+        xyz="0 0 0"
+        rpy="0 0 0" />
+      <geometry>
+        <mesh
+          filename="package://gummi_rightbase_$(env ROS_GUMMI_RIGHTBASE)/meshes/upperarm_biceps_pulley.STL" />
       </geometry>
     </collision>
@@ -406,19 +406,19 @@
       <geometry>
         <mesh
-          filename="package://gummi_base_$(env ROS_GUMMI_BASE)/meshes/upperarm_triceps_pulley.STL" />
-      </geometry>
-      <material
-        name="">
-        <color
-          rgba="0.79216 0.81961 0.93333 1" />
-      </material>
-    </visual>
-    <collision>
-      <origin
-        xyz="0 0 0"
-        rpy="0 0 0" />
-      <geometry>
-        <mesh
-          filename="package://gummi_base_$(env ROS_GUMMI_BASE)/meshes/upperarm_triceps_pulley.STL" />
+          filename="package://gummi_rightbase_$(env ROS_GUMMI_RIGHTBASE)/meshes/upperarm_triceps_pulley.STL" />
+      </geometry>
+      <material
+        name="">
+        <color
+          rgba="0.79216 0.81961 0.93333 1" />
+      </material>
+    </visual>
+    <collision>
+      <origin
+        xyz="0 0 0"
+        rpy="0 0 0" />
+      <geometry>
+        <mesh
+          filename="package://gummi_rightbase_$(env ROS_GUMMI_RIGHTBASE)/meshes/upperarm_triceps_pulley.STL" />
       </geometry>
     </collision>
@@ -462,19 +462,19 @@
       <geometry>
         <mesh
-          filename="package://gummi_base_$(env ROS_GUMMI_BASE)/meshes/shoulder_roll_top_pulley.STL" />
-      </geometry>
-      <material
-        name="">
-        <color
-          rgba="0.79216 0.81961 0.93333 1" />
-      </material>
-    </visual>
-    <collision>
-      <origin
-        xyz="0 0 0"
-        rpy="0 0 0" />
-      <geometry>
-        <mesh
-          filename="package://gummi_base_$(env ROS_GUMMI_BASE)/meshes/shoulder_roll_top_pulley.STL" />
+          filename="package://gummi_rightbase_$(env ROS_GUMMI_RIGHTBASE)/meshes/shoulder_roll_top_pulley.STL" />
+      </geometry>
+      <material
+        name="">
+        <color
+          rgba="0.79216 0.81961 0.93333 1" />
+      </material>
+    </visual>
+    <collision>
+      <origin
+        xyz="0 0 0"
+        rpy="0 0 0" />
+      <geometry>
+        <mesh
+          filename="package://gummi_rightbase_$(env ROS_GUMMI_RIGHTBASE)/meshes/shoulder_roll_top_pulley.STL" />
       </geometry>
     </collision>
@@ -515,19 +515,19 @@
       <geometry>
         <mesh
-          filename="package://gummi_base_$(env ROS_GUMMI_BASE)/meshes/shoulder_roll_bottom_pulley.STL" />
-      </geometry>
-      <material
-        name="">
-        <color
-          rgba="0.79216 0.81961 0.93333 1" />
-      </material>
-    </visual>
-    <collision>
-      <origin
-        xyz="0 0 0"
-        rpy="0 0 0" />
-      <geometry>
-        <mesh
-          filename="package://gummi_base_$(env ROS_GUMMI_BASE)/meshes/shoulder_roll_bottom_pulley.STL" />
+          filename="package://gummi_rightbase_$(env ROS_GUMMI_RIGHTBASE)/meshes/shoulder_roll_bottom_pulley.STL" />
+      </geometry>
+      <material
+        name="">
+        <color
+          rgba="0.79216 0.81961 0.93333 1" />
+      </material>
+    </visual>
+    <collision>
+      <origin
+        xyz="0 0 0"
+        rpy="0 0 0" />
+      <geometry>
+        <mesh
+          filename="package://gummi_rightbase_$(env ROS_GUMMI_RIGHTBASE)/meshes/shoulder_roll_bottom_pulley.STL" />
       </geometry>
     </collision>
@@ -571,19 +571,19 @@
       <geometry>
         <mesh
-          filename="package://gummi_base_$(env ROS_GUMMI_BASE)/meshes/shoulder_pitch_front_pulley.STL" />
-      </geometry>
-      <material
-        name="">
-        <color
-          rgba="0.79216 0.81961 0.93333 1" />
-      </material>
-    </visual>
-    <collision>
-      <origin
-        xyz="0 0 0"
-        rpy="0 0 0" />
-      <geometry>
-        <mesh
-          filename="package://gummi_base_$(env ROS_GUMMI_BASE)/meshes/shoulder_pitch_front_pulley.STL" />
+          filename="package://gummi_rightbase_$(env ROS_GUMMI_RIGHTBASE)/meshes/shoulder_pitch_front_pulley.STL" />
+      </geometry>
+      <material
+        name="">
+        <color
+          rgba="0.79216 0.81961 0.93333 1" />
+      </material>
+    </visual>
+    <collision>
+      <origin
+        xyz="0 0 0"
+        rpy="0 0 0" />
+      <geometry>
+        <mesh
+          filename="package://gummi_rightbase_$(env ROS_GUMMI_RIGHTBASE)/meshes/shoulder_pitch_front_pulley.STL" />
       </geometry>
     </collision>
@@ -624,19 +624,19 @@
       <geometry>
         <mesh
-          filename="package://gummi_base_$(env ROS_GUMMI_BASE)/meshes/shoulder_pitch_back_pulley.STL" />
-      </geometry>
-      <material
-        name="">
-        <color
-          rgba="0.79216 0.81961 0.93333 1" />
-      </material>
-    </visual>
-    <collision>
-      <origin
-        xyz="0 0 0"
-        rpy="0 0 0" />
-      <geometry>
-        <mesh
-          filename="package://gummi_base_$(env ROS_GUMMI_BASE)/meshes/shoulder_pitch_back_pulley.STL" />
+          filename="package://gummi_rightbase_$(env ROS_GUMMI_RIGHTBASE)/meshes/shoulder_pitch_back_pulley.STL" />
+      </geometry>
+      <material
+        name="">
+        <color
+          rgba="0.79216 0.81961 0.93333 1" />
+      </material>
+    </visual>
+    <collision>
+      <origin
+        xyz="0 0 0"
+        rpy="0 0 0" />
+      <geometry>
+        <mesh
+          filename="package://gummi_rightbase_$(env ROS_GUMMI_RIGHTBASE)/meshes/shoulder_pitch_back_pulley.STL" />
       </geometry>
     </collision>
