Commit message: it moves

File: xacro/gummi_description_base.urdf.xacro (robot description, xacro)
@@ -2,5 +2,5 @@
 <robot>
   <link
-    name="base_link">
+    name="right_base_link">
     <inertial>
       <origin
@@ -88,5 +88,5 @@
       rpy="0 0 0" />
     <parent
-      link="base_link" />
+      link="right_base_link" />
     <child
       link="shoulder_preroll" />

File: xacro/gummi_right.urdf.xacro (robot description, xacro)
@@ -4,10 +4,3 @@
 <xacro:include filename="$(env GUMMI_RIGHTBASEPATH)/xacro/gummi_description_base.urdf.xacro" />
 <xacro:include filename="$(env GUMMI_RIGHTEEPATH)/xacro/gummi_description_ee.urdf.xacro" />
-<link name="base_link"/>
-<joint name="rightbase_displacement" type="fixed">
-  <origin rpy="0 0 0" xyz="0.2 0 0"/>
-  <parent link="base_link"/>
-  <child link="right_base_link"/>
-  <axis xyz="0 0 0"/>
-</joint>
 </robot>
