Commit message: make it right

File: xacro/gummi_base.srdf.xacro (robot description, xacro)
@@ -4,47 +4,47 @@
       <!-- <chain base_link="base_link" tip_link="right_hand" /> -->
 <xacro:macro name="group_right_arm_base">
-  <joint name="shoulder_yaw" />
-  <joint name="shoulder_roll" />
-  <joint name="shoulder_pitch" />
-  <joint name="upperarm_roll" />
-  <joint name="elbow" />
-  <joint name="fastswitch" />
+  <joint name="right/shoulder_yaw" />
+  <joint name="right/shoulder_roll" />
+  <joint name="right/shoulder_pitch" />
+  <joint name="right/upperarm_roll" />
+  <joint name="right/elbow" />
+  <joint name="right/fastswitch" />
 </xacro:macro>
 <xacro:macro name="group_state_right_arm_base">
-  <joint name="shoulder_pitch" value="0" />
-  <joint name="shoulder_roll" value="0" />
-  <joint name="shoulder_yaw" value="0" />
-  <joint name="upperarm_roll" value="0" />
-  <joint name="elbow" value="0" />
+  <joint name="right/shoulder_pitch" value="0" />
+  <joint name="right/shoulder_roll" value="0" />
+  <joint name="right/shoulder_yaw" value="0" />
+  <joint name="right/upperarm_roll" value="0" />
+  <joint name="right/elbow" value="0" />
 </xacro:macro>
 <xacro:macro name="virtual_joints_base">
   <!--VIRTUAL JOINT: Purpose: this element defines a virtual joint between a robot link and an external frame of reference (considered fixed with respect to the robot)-->
-  <virtual_joint name="virtual_joint" type="fixed" parent_frame="map" child_link="base_link" />
+  <virtual_joint name="virtual_joint" type="fixed" parent_frame="map" child_link="right/base_link" />
 </xacro:macro>
 <xacro:macro name="disable_collisions_base">
   <!--DISABLE COLLISIONS: By default it is assumed that any link of the robot could potentially come into collision with any other link in the robot. This tag disables collision checking between a specified pair of links. -->
-  <disable_collisions link1="base_link" link2="shoulder" reason="Never" />
-  <disable_collisions link1="base_link" link2="shoulder_preroll" reason="Adjacent" />
-  <disable_collisions link1="base_link" link2="upperarm" reason="Never" />
-  <disable_collisions link1="base_link" link2="upperarm_preroll" reason="Never" />
-  <disable_collisions link1="shoulder" link2="shoulder_preroll" reason="Adjacent" />
-  <disable_collisions link1="shoulder" link2="upperarm" reason="Never" />
-  <disable_collisions link1="shoulder" link2="upperarm_preroll" reason="Adjacent" />
-  <disable_collisions link1="shoulder_preroll" link2="upperarm" reason="Never" />
-  <disable_collisions link1="shoulder_preroll" link2="upperarm_preroll" reason="Never" />
-  <disable_collisions link1="upperarm" link2="upperarm_preroll" reason="Adjacent" />
+  <disable_collisions link1="right/base_link" link2="right/shoulder" reason="Never" />
+  <disable_collisions link1="right/base_link" link2="right/shoulder_preroll" reason="Adjacent" />
+  <disable_collisions link1="right/base_link" link2="right/upperarm" reason="Never" />
+  <disable_collisions link1="right/base_link" link2="right/upperarm_preroll" reason="Never" />
+  <disable_collisions link1="right/shoulder" link2="right/shoulder_preroll" reason="Adjacent" />
+  <disable_collisions link1="right/shoulder" link2="right/upperarm" reason="Never" />
+  <disable_collisions link1="right/shoulder" link2="right/upperarm_preroll" reason="Adjacent" />
+  <disable_collisions link1="right/shoulder_preroll" link2="right/upperarm" reason="Never" />
+  <disable_collisions link1="right/shoulder_preroll" link2="right/upperarm_preroll" reason="Never" />
+  <disable_collisions link1="right/upperarm" link2="right/upperarm_preroll" reason="Adjacent" />
 </xacro:macro>
 <xacro:macro name="disable_collisions_mixed">
   <!--MIXED DISABLE COLLISIONS FOR BASE EE COLISIONS: set by hand or remove! -->
-  <disable_collisions link1="base_link" link2="lowerarm_preroll_u" reason="Never" />
-  <disable_collisions link1="lowerarm" link2="shoulder" reason="Never" />
-  <disable_collisions link1="lowerarm" link2="shoulder_preroll" reason="Never" />
-  <disable_collisions link1="lowerarm" link2="upperarm" reason="Never" />
-  <disable_collisions link1="lowerarm" link2="upperarm_preroll" reason="Never" />
-  <disable_collisions link1="lowerarm_preroll_u" link2="shoulder" reason="Never" />
-  <disable_collisions link1="lowerarm_preroll_u" link2="shoulder_preroll" reason="Never" />
-  <disable_collisions link1="lowerarm_preroll_u" link2="upperarm" reason="Adjacent" />
-  <disable_collisions link1="lowerarm_preroll_u" link2="upperarm_preroll" reason="Never" />
-  <disable_collisions link1="lowerarm_preroll_u" link2="lowerarm_preroll_d" reason="Adjacent" />
+  <disable_collisions link1="right/base_link" link2="right/lowerarm_preroll_u" reason="Never" />
+  <disable_collisions link1="right/lowerarm" link2="right/shoulder" reason="Never" />
+  <disable_collisions link1="right/lowerarm" link2="right/shoulder_preroll" reason="Never" />
+  <disable_collisions link1="right/lowerarm" link2="right/upperarm" reason="Never" />
+  <disable_collisions link1="right/lowerarm" link2="right/upperarm_preroll" reason="Never" />
+  <disable_collisions link1="right/lowerarm_preroll_u" link2="right/shoulder" reason="Never" />
+  <disable_collisions link1="right/lowerarm_preroll_u" link2="right/shoulder_preroll" reason="Never" />
+  <disable_collisions link1="right/lowerarm_preroll_u" link2="right/upperarm" reason="Adjacent" />
+  <disable_collisions link1="right/lowerarm_preroll_u" link2="right/upperarm_preroll" reason="Never" />
+  <disable_collisions link1="right/lowerarm_preroll_u" link2="right/lowerarm_preroll_d" reason="Adjacent" />
 </xacro:macro>
 </robot>

File: xacro/gummi_description.urdf.xacro (robot description, xacro)
@@ -8,5 +8,5 @@
   <origin rpy="0 0 0" xyz="0.2 0 0"/>
   <parent link="base_link"/>
-  <child link="right_base_link"/>
+  <child link="right/base_link"/>
   <axis xyz="0 0 0"/>
 </joint>

File: xacro/gummi_description_base.urdf.xacro (robot description, xacro)
@@ -2,5 +2,5 @@
 <robot>
   <link
-    name="right_base_link">
+    name="right/base_link">
     <inertial>
       <origin
@@ -42,5 +42,5 @@
   </link>
   <link
-    name="shoulder_preroll">
+    name="right/shoulder_preroll">
     <inertial>
       <origin
@@ -82,5 +82,5 @@
   </link>
   <joint
-    name="shoulder_yaw"
+    name="right/shoulder_yaw"
     type="revolute">
     <origin
@@ -88,7 +88,7 @@
       rpy="0 0 0" />
     <parent
-      link="right_base_link" />
-    <child
-      link="shoulder_preroll" />
+      link="right/base_link" />
+    <child
+      link="right/shoulder_preroll" />
     <axis
       xyz="0 0 1" />
@@ -100,5 +100,5 @@
   </joint>
   <link
-    name="shoulder">
+    name="right/shoulder">
     <inertial>
       <origin
@@ -140,5 +140,5 @@
   </link>
   <joint
-    name="shoulder_roll"
+    name="right/shoulder_roll"
     type="revolute">
     <origin
@@ -146,7 +146,7 @@
       rpy="0 0 0" />
     <parent
-      link="shoulder_preroll" />
-    <child
-      link="shoulder" />
+      link="right/shoulder_preroll" />
+    <child
+      link="right/shoulder" />
     <axis
       xyz="0 -1 0" />
@@ -158,5 +158,5 @@
   </joint>
   <link
-    name="upperarm_preroll">
+    name="right/upperarm_preroll">
     <inertial>
       <origin
@@ -198,5 +198,5 @@
   </link>
   <joint
-    name="shoulder_pitch"
+    name="right/shoulder_pitch"
     type="revolute">
     <origin
@@ -204,7 +204,7 @@
       rpy="0 0 0" />
     <parent
-      link="shoulder" />
-    <child
-      link="upperarm_preroll" />
+      link="right/shoulder" />
+    <child
+      link="right/upperarm_preroll" />
     <axis
       xyz="-1 0 0" />
@@ -216,5 +216,5 @@
   </joint>
   <link
-    name="upperarm">
+    name="right/upperarm">
     <inertial>
       <origin
@@ -256,5 +256,5 @@
   </link>
   <joint
-    name="upperarm_roll"
+    name="right/upperarm_roll"
     type="revolute">
     <origin
@@ -262,7 +262,7 @@
       rpy="0 0 0" />
     <parent
-      link="upperarm_preroll" />
-    <child
-      link="upperarm" />
+      link="right/upperarm_preroll" />
+    <child
+      link="right/upperarm" />
     <axis
       xyz="0 0 -1" />
@@ -274,5 +274,5 @@
   </joint>
   <link
-    name="lowerarm_preroll_u">
+    name="right/lowerarm_preroll_u">
     <inertial>
       <origin
@@ -314,5 +314,5 @@
   </link>
   <joint
-    name="elbow"
+    name="right/elbow"
     type="revolute">
     <origin
@@ -320,7 +320,7 @@
       rpy="0 0 0" />
     <parent
-      link="upperarm" />
-    <child
-      link="lowerarm_preroll_u" />
+      link="right/upperarm" />
+    <child
+      link="right/lowerarm_preroll_u" />
     <axis
       xyz="0 -1 0" />
@@ -332,5 +332,5 @@
   </joint>
   <link
-    name="upperarm_biceps_pulley">
+    name="right/upperarm_biceps_pulley">
     <inertial>
       <origin
@@ -372,5 +372,5 @@
   </link>
   <joint
-    name="upperarm_biceps_pulley_joint"
+    name="right/upperarm_biceps_pulley_joint"
     type="fixed">
     <origin
@@ -378,12 +378,12 @@
       rpy="0 0 0" />
     <parent
-      link="upperarm" />
-    <child
-      link="upperarm_biceps_pulley" />
+      link="right/upperarm" />
+    <child
+      link="right/upperarm_biceps_pulley" />
     <axis
       xyz="0 0 0" />
   </joint>
   <link
-    name="upperarm_triceps_pulley">
+    name="right/upperarm_triceps_pulley">
     <inertial>
       <origin
@@ -425,5 +425,5 @@
   </link>
   <joint
-    name="upperarm_triceps_pulley_joint"
+    name="right/upperarm_triceps_pulley_joint"
     type="fixed">
     <origin
@@ -431,7 +431,7 @@
       rpy="0 0 0" />
     <parent
-      link="upperarm" />
-    <child
-      link="upperarm_triceps_pulley" />
+      link="right/upperarm" />
+    <child
+      link="right/upperarm_triceps_pulley" />
     <axis
       xyz="-1 0 0" />
@@ -441,5 +441,5 @@
   </joint>
   <link
-    name="shoulder_roll_top_pulley">
+    name="right/shoulder_roll_top_pulley">
     <inertial>
       <origin
@@ -481,5 +481,5 @@
   </link>
   <joint
-    name="shoulder_roll_top_pulley_joint"
+    name="right/shoulder_roll_top_pulley_joint"
     type="fixed">
     <origin
@@ -487,12 +487,12 @@
       rpy="0 0 0" />
     <parent
-      link="shoulder" />
-    <child
-      link="shoulder_roll_top_pulley" />
+      link="right/shoulder" />
+    <child
+      link="right/shoulder_roll_top_pulley" />
     <axis
       xyz="0 0 0" />
   </joint>
   <link
-    name="shoulder_roll_bottom_pulley">
+    name="right/shoulder_roll_bottom_pulley">
     <inertial>
       <origin
@@ -534,5 +534,5 @@
   </link>
   <joint
-    name="shoulder_roll_bottom_pulley"
+    name="right/shoulder_roll_bottom_pulley"
     type="fixed">
     <origin
@@ -540,7 +540,7 @@
       rpy="0 0 0" />
     <parent
-      link="shoulder" />
-    <child
-      link="shoulder_roll_bottom_pulley" />
+      link="right/shoulder" />
+    <child
+      link="right/shoulder_roll_bottom_pulley" />
     <axis
       xyz="0 0 -1" />
@@ -550,5 +550,5 @@
   </joint>
   <link
-    name="shoulder_pitch_front_pulley">
+    name="right/shoulder_pitch_front_pulley">
     <inertial>
       <origin
@@ -590,5 +590,5 @@
   </link>
   <joint
-    name="shoulder_pitch_pulley_front_joint"
+    name="right/shoulder_pitch_pulley_front_joint"
     type="fixed">
     <origin
@@ -596,12 +596,12 @@
       rpy="0 0 0" />
     <parent
-      link="shoulder_preroll" />
-    <child
-      link="shoulder_pitch_front_pulley" />
+      link="right/shoulder_preroll" />
+    <child
+      link="right/shoulder_pitch_front_pulley" />
     <axis
       xyz="0 0 0" />
   </joint>
   <link
-    name="shoulder_pitch_back_pulley">
+    name="right/shoulder_pitch_back_pulley">
     <inertial>
       <origin
@@ -643,5 +643,5 @@
   </link>
   <joint
-    name="shoulder_pitch_back_pulley_joint"
+    name="right/shoulder_pitch_back_pulley_joint"
     type="fixed">
     <origin
@@ -649,7 +649,7 @@
       rpy="0 0 0" />
     <parent
-      link="shoulder_preroll" />
-    <child
-      link="shoulder_pitch_back_pulley" />
+      link="right/shoulder_preroll" />
+    <child
+      link="right/shoulder_pitch_back_pulley" />
     <axis
       xyz="0 0 0" />
